File: kicad/twitch treatbot feather carrier.kicad_pcb (KiCad board)
At the start: 4 copper layers, 59.8 x 58.1 mm, 76 parts, among them J1 128x64 OLED, J2 Quiic MP3 Trigger [CHECK FOOT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, J3 M2, J4 M1, J5 +12V_IN, J6 NEO_Signal, J7 +5V_IN, Q1 BSS138, SW1 ESP RESET, SW2 Wiggle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

Commit message: rev1-to-fab
Parts:
- added C6: 10u, Capacitor_SMD:C_0805_2012Metric, F.Cu at (58.5, 85.6)
- added REF**: ESD-Logo_6.6x6mm_SilkScreen, Symbol:ESD-Logo_6.6x6mm_SilkScreen, B.Cu at (107.1, 109.3)
- added REF**: KiCad-Logo2_5mm_SilkScreen, Symbol:KiCad-Logo2_5mm_SilkScreen, B.Cu at (61.0, 107.2)
- added REF**: OSHW-Symbol_6.7x6mm_SilkScreen, Symbol:OSHW-Symbol_6.7x6mm_SilkScreen, B.Cu at (60.5, 98.9)
- added kibuzzard-622633E5: G***, kibuzzard-622633E5, F.Cu at (109.8, 102.1)
- added kibuzzard-622633FA: G***, kibuzzard-622633FA, F.Cu at (109.8, 92.0)
- added kibuzzard-62263418: G***, kibuzzard-62263418, F.Cu at (109.8, 97.2)
- added kibuzzard-62263431: G***, kibuzzard-62263431, F.Cu at (109.8, 87.0)
- added kibuzzard-62263481: G***, kibuzzard-62263481, F.Cu at (105.8, 57.1)
- added kibuzzard-62263491: G***, kibuzzard-62263491, F.Cu at (93.1, 57.0)
- added kibuzzard-622642D3: G***, kibuzzard-622642D3, F.Cu at (63.1, 84.3)
- added kibuzzard-622647CC: G***, kibuzzard-622647CC, B.Cu at (60.9, 90.4)
- added svg2mod: G***, My Libraries:BE10v2, B.Cu at (70.2, 72.9)
- moved kibuzzard-622633E5 10.9 mm to (108.2, 102.3)
- moved kibuzzard-622633FA 10.9 mm to (108.2, 92.2)
- moved kibuzzard-62263418 10.9 mm to (108.2, 97.4)
- moved kibuzzard-62263431 10.9 mm to (108.2, 87.2)
- moved R1 0.13 mm to (58.5, 83.2)
Connections:
- A1 pad 27: +5V -> Net-(A1-Pad27)
- R1 pad 2: GND -> Net-(A1-Pad27)
Routing:
- net Net-(A1-Pad27): track 0.00 -> 8.05 mm
- net +5V: track 46.3 -> 46.2 mm, vias 4 -> 5
Other:
- board text added: "Delay for EN"
