File: kicad/twitch treatbot feather carrier.kicad_sch (KiCad schematic)
At the start: 40 parts, among them J1 128x64 OLED, J2 Quiic MP3 Trigger [CHECK FOOT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, J3 M2, J4 M1, J5 +12V_IN, J6 NEO_Signal, J7 +5V_IN, Q1 BSS138, SW1 ESP RESET, SW2 Wiggle, U1 TMC2208_BREAKOUT

Commit message: rev1-to-fab
Parts:
- added C6: 10u, Capacitor_SMD:C_0805_2012Metric, symbol My Library:C_0805
Connections:
- net +5V: no longer A1.27 (EN)
- net GND: now also C6.2; no longer R1.2
- new net: A1.27 (EN), C6.1, R1.2
Other:
- moved on the sheet: R1
Changed lines of the file:
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@@
   (junction (at 165.735 125.73) (diameter 0) (color 0 0 0 0)
   )
+  (junction (at 105.41 62.23) (diameter 0) (color 0 0 0 0)
+  )
   (junction (at 134.62 125.73) (diameter 0) (color 0 0 0 0)
   )
@@
   )
   (junction (at 177.8 125.73) (diameter 0) (color 0 0 0 0)
-  )
-  (junction (at 87.63 59.69) (diameter 0) (color 0 0 0 0)
   )
   (junction (at 143.51 116.205) (diameter 0) (color 0 0 0 0)
@@
     (stroke (width 0) (type default) (color 0 0 0 0))
   )
-  (wire (pts (xy 87.63 59.69) (xy 87.63 60.96))
+  (wire (pts (xy 87.63 59.69) (xy 87.63 62.23))
     (stroke (width 0) (type default) (color 0 0 0 0))
   )
@@
     (stroke (width 0) (type default) (color 0 0 0 0))
   )
+  (wire (pts (xy 105.41 62.23) (xy 105.41 63.5))
+    (stroke (width 0) (type default) (color 0 0 0 0))
+  )
   (wire (pts (xy 160.02 46.355) (xy 165.735 46.355))
     (stroke (width 0) (type default) (color 0 0 0 0))
@@
     (stroke (width 0) (type default) (color 0 0 0 0))
   )
+  (wire (pts (xy 105.41 60.96) (xy 105.41 62.23))
+    (stroke (width 0) (type default) (color 0 0 0 0))
+  )
   (wire (pts (xy 129.54 29.21) (xy 135.255 29.21))
     (stroke (width 0) (type default) (color 0 0 0 0))
@@
   )
   (wire (pts (xy 165.735 125.73) (xy 161.925 125.73))
+    (stroke (width 0) (type default) (color 0 0 0 0))
+  )
+  (wire (pts (xy 87.63 62.23) (xy 105.41 62.23))
     (stroke (width 0) (type default) (color 0 0 0 0))
   )
@@
     (pin "1")
   )
-  (symbol (lib_id "power:+5V") (at 87.63 59.69 0) (unit 1)
+  (symbol (lib_id "power:+5V") (at 105.41 55.88 0) (unit 1)
     (in_bom yes) (on_board yes)
-    (property "Reference" "#PWR0110" (id 0) (at 87.63 63.5 0)
-      (effects (font (size 1.27 1.27)) hide)
-    )
-    (property "Value" "+5V" (id 1) (at 87.63 54.61 0))
-    (property "Footprint" "" (id 2) (at 87.63 59.69 0)
-      (effects (font (size 1.27 1.27)) hide)
-    )
-    (property "Datasheet" "" (id 3) (at 87.63 59.69 0)
+    (property "Reference" "#PWR0110" (id 0) (at 105.41 59.69 0)
+      (effects (font (size 1.27 1.27)) hide)
+    )
+    (property "Value" "+5V" (id 1) (at 105.41 50.8 0))
+    (property "Footprint" "" (id 2) (at 105.41 55.88 0)
+      (effects (font (size 1.27 1.27)) hide)
+    )
+    (property "Datasheet" "" (id 3) (at 105.41 55.88 0)
       (effects (font (size 1.27 1.27)) hide)
     )
@@
     (pin "9")
   )
+  (symbol (lib_id "My Library:C_0805") (at 105.41 66.04 0) (unit 1)
+    (in_bom yes) (on_board yes) (fields_autoplaced)
+    (property "Reference" "C6" (id 0) (at 108.585 64.7762 0)
+      (effects (font (size 1.27 1.27)) (justify left))
+    )
+    (property "Value" "10u" (id 1) (at 108.585 67.3162 0)
+      (effects (font (size 1.27 1.27)) (justify left))
+    )
+    (property "Footprint" "Capacitor_SMD:C_0805_2012Metric" (id 2) (at 105.41 66.04 0)
+      (effects (font (size 1.27 1.27)) hide)
+    )
+    (property "Datasheet" "~" (id 3) (at 105.41 66.04 0)
+      (effects (font (size 1.27 1.27)) hide)
+    )
+    (pin "1")
+    (pin "2")
+  )
   (symbol (lib_id "Connector_Generic:Conn_01x02") (at 140.335 55.88 0) (unit 1)
     (in_bom yes) (on_board yes) (fields_autoplaced)
@@
     (pin "1")
   )
-  (symbol (lib_id "power:GND") (at 87.63 66.04 0) (unit 1)
-    (in_bom yes) (on_board yes) (fields_autoplaced)
-    (property "Reference" "#PWR0111" (id 0) (at 87.63 72.39 0)
-      (effects (font (size 1.27 1.27)) hide)
-    )
-    (property "Value" "GND" (id 1) (at 87.63 71.12 0))
-    (property "Footprint" "" (id 2) (at 87.63 66.04 0)
-      (effects (font (size 1.27 1.27)) hide)
-    )
-    (property "Datasheet" "" (id 3) (at 87.63 66.04 0)
+  (symbol (lib_id "power:GND") (at 105.41 68.58 0) (unit 1)
+    (in_bom yes) (on_board yes) (fields_autoplaced)
+    (property "Reference" "#PWR0111" (id 0) (at 105.41 74.93 0)
+      (effects (font (size 1.27 1.27)) hide)
+    )
+    (property "Value" "GND" (id 1) (at 105.41 73.66 0))
+    (property "Footprint" "" (id 2) (at 105.41 68.58 0)
+      (effects (font (size 1.27 1.27)) hide)
+    )
+    (property "Datasheet" "" (id 3) (at 105.41 68.58 0)
       (effects (font (size 1.27 1.27)) hide)
     )
@@
     (pin "3")
   )
-  (symbol (lib_id "My Library:R_0805") (at 87.63 63.5 0) (unit 1)
-    (in_bom yes) (on_board yes) (fields_autoplaced)
-    (property "Reference" "R1" (id 0) (at 89.535 62.2299 0)
-      (effects (font (size 1.27 1.27)) (justify left))
-    )
-    (property "Value" "10k" (id 1) (at 89.535 64.7699 0)
-      (effects (font (size 1.27 1.27)) (justify left))
-    )
-    (property "Footprint" "Resistor_SMD:R_0805_2012Metric" (id 2) (at 87.63 63.5 0)
-      (effects (font (size 1.27 1.27)) hide)
-    )
-    (property "Datasheet" "~" (id 3) (at 87.63 63.5 0)
+  (symbol (lib_id "My Library:R_0805") (at 105.41 58.42 0) (unit 1)
+    (in_bom yes) (on_board yes) (fields_autoplaced)
+    (property "Reference" "R1" (id 0) (at 107.315 57.1499 0)
+      (effects (font (size 1.27 1.27)) (justify left))
+    )
+    (property "Value" "10k" (id 1) (at 107.315 59.6899 0)
+      (effects (font (size 1.27 1.27)) (justify left))
+    )
+    (property "Footprint" "Resistor_SMD:R_0805_2012Metric" (id 2) (at 105.41 58.42 0)
+      (effects (font (size 1.27 1.27)) hide)
+    )
+    (property "Datasheet" "~" (id 3) (at 105.41 58.42 0)
       (effects (font (size 1.27 1.27)) hide)
     )
@@
       (reference "C5") (unit 1) (value "1u") (footprint "Capacitor_SMD:C_0805_2012Metric")
     )
+    (path "/58a97278-0dca-4489-85d8-90f2ed606d8c"
+      (reference "C6") (unit 1) (value "10u") (footprint "Capacitor_SMD:C_0805_2012Metric")
+    )
     (path "/2e3714ea-d9f6-4749-8d86-b3cc39ce5e7a"

Commit message: added NC to existing pins and made notes after reviewing built design. IO15 was a lousy pick for the Wiggle button.
Connections:
- no-connect marks 12 -> 14
Other:
- note added: "IO15 is used during boot, it shouldn't be used as an input. (Could have been an output)"
- note removed: "Move STEP signal from IO0 to IO15. IO0 should have an on-board led"
Changed lines of the file:
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@@
   (junction (at 143.51 116.205) (diameter 0) (color 0 0 0 0)
   )
+  (no_connect (at 55.88 54.61))
   (no_connect (at 81.28 57.15))
   (no_connect (at 81.28 67.31))
+  (no_connect (at 55.88 52.07))
   (no_connect (at 55.88 62.23))
   (no_connect (at 55.88 64.77))
@@
     (stroke (width 0) (type default) (color 0 0 0 0))
   )
-  (wire (pts (xy 44.45 54.61) (xy 55.88 54.61))
-    (stroke (width 0) (type default) (color 0 0 0 0))
-  )
   (wire (pts (xy 129.54 44.45) (xy 135.255 44.45))
     (stroke (width 0) (type default) (color 0 0 0 0))
@@
     (stroke (width 0) (type default) (color 0 0 0 0))
   )
-  (wire (pts (xy 44.45 52.07) (xy 55.88 52.07))
-    (stroke (width 0) (type default) (color 0 0 0 0))
-  )
   (wire (pts (xy 156.845 116.205) (xy 143.51 116.205))
     (stroke (width 0) (type default) (color 0 0 0 0))
@@
     (stroke (width 0) (type default) (color 0 0 0 0))
   )
-  (text "Move STEP signal from IO0 to IO15.\nIO0 should have an on-board led"
-    (at 31.75 39.37 0)
+  (text "IO15 is used during boot, it shouldn't be used as an input.\n\n(Could have been an output)"
+    (at 19.685 43.18 0)
     (effects (font (size 1.27 1.27)) (justify left bottom))
   )
